File: PMOD_MEM.kicad_sch (KiCad schematic)
At the start: 6 parts, among them IC1 W25Q16JVSNIQ, U1 CAT24M01W

Commit message: Fixed library paths
Parts:
- C1: footprint (none) -> Capacitor_SMD:C_0805_2012Metric
- R1, R2: footprint (none) -> Resistor_SMD:R_0805_2012Metric
Changed lines of the file:
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@@
     (property "Reference" "R1" (id 0) (at 164.592 64.77 90))
     (property "Value" "1K" (id 1) (at 162.56 64.77 90))
-    (property "Footprint" "" (id 2) (at 160.782 64.77 90)
+    (property "Footprint" "Resistor_SMD:R_0805_2012Metric" (id 2) (at 160.782 64.77 90)
       (effects (font (size 1.27 1.27)) hide)
     )
@@
       (effects (font (size 1.27 1.27)) (justify left))
     )
-    (property "Footprint" "" (id 2) (at 107.6452 101.6 0)
+    (property "Footprint" "Capacitor_SMD:C_0805_2012Metric" (id 2) (at 107.6452 101.6 0)
       (effects (font (size 1.27 1.27)) hide)
     )
@@
       (effects (font (size 1.27 1.27)) (justify left))
     )
-    (property "Footprint" "" (id 2) (at 164.592 64.77 90)
+    (property "Footprint" "Resistor_SMD:R_0805_2012Metric" (id 2) (at 164.592 64.77 90)
       (effects (font (size 1.27 1.27)) hide)
     )
